File: pcb/Ai_Breakout_OLED-0.96.sch (EAGLE design)
At the start: 14 parts, among them J1 2X04, M1 STAND-OFF, M2 STAND-OFF, M3 STAND-OFF, M4 STAND-OFF, U1 UG-2864HSWEG01

Commit message: routing done
Parts:
- removed JP1: 1X07, Ai_Connectors:1X07
- added C1, C2: 10uF, Ai_Passives:CAP0603
- added IC1: 74HCT245MTC, Ai_IC:74HCT245MTC
- added J2: 1X08, Ai_Connectors:1X08
- added JS1, JS2: 1X02-SJ-NO, Ai_Connectors:1X02-SJ-NO
- added R1: 10K, Ai_Passives:RES0603
- added U2: MIC5205-3.3, Ai_Power:MIC5205-3.3
- C5: value 10uF -> 2.2uF
- C8: value 2.2uF -> 10uF
Connections:
- new net CS_IN: IC1.A5, J1.5, J2.5
- new net D0/SCLK/SCK_IN: IC1.A2, J1.2, J2.2
- new net D1/MOSI/SDA1_IN: IC1.A1, J1.1, J2.1
- new net DC/SA0_IN: IC1.A3, J1.3, J2.3
- new net I2C_EN: JS2.1, R1.2, U1.BS1
- new net N$8: JS1.2, U1.D2/I2C_SDA
- new net RST_IN: IC1.A4, J1.4, J2.4
- new net VIN: C1.2, J1.7, J2.7, U2.EN, U2.IN
- net 3V3: now also C2.2, C5.2, IC1.DIR, IC1.VCC, J1.6, J2.6, JS2.2, U2.OUT; no longer C7.2, JP1.6
- net CS_3V3: now also IC1.B5; no longer JP1.5
- net D0/SCLK/SCK_3V3: now also IC1.B2; no longer JP1.2
- net D1/MOSI/SDA1_3V3: now also IC1.B1, JS1.1; no longer JP1.1
- net DC/SA0_3V3: now also IC1.B3; no longer JP1.3
- net GND: now also C1.1, C2.1, IC1.!OE, IC1.GND, J1.8, J2.8, R1.1, U2.GND; no longer JP1.7, U1.BS1
- net N$11: now also C8.2; no longer C5.2
- net N$12: now also C7.2; no longer C8.2
- net RST_3V3: now also IC1.B4; no longer JP1.4
Other:
- moved on the sheet: C3, C4, C5, C6, C7, C8, R3

Commit message: ready for fabrication
Parts:
- added U$15, U$16: AI-LOGOXS, Ai_Miscellany:AI-LOGOXS
Connections:
- net CS_3V3: now also U1.!CS; no longer U1./CS
- net RST_3V3: now also U1.!RST; no longer U1./RES
Changed lines of the file:
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@@
 <part name="U$12" library="Ai_Power" deviceset="3V3" device=""/>
 <part name="U$14" library="Ai_Power" deviceset="GND" device=""/>
+<part name="U$15" library="Ai_Miscellany" deviceset="AI-LOGO" device="XS"/>
+<part name="U$16" library="Ai_Miscellany" deviceset="AI-LOGO" device="XS"/>
 </parts>
 <sheets>
@@
 <instance part="U$12" gate="G$1" x="49.53" y="59.69"/>
 <instance part="U$14" gate="GND" x="80.01" y="26.67"/>
+<instance part="U$15" gate="G$1" x="123.19" y="16.51"/>
+<instance part="U$16" gate="G$1" x="123.19" y="16.51"/>
 </instances>
 <busses>
@@
 <wire x1="110.49" y1="152.4" x2="110.49" y2="134.62" width="0.1524" layer="91"/>
 <junction x="110.49" y="134.62"/>
+<junction x="110.49" y="88.9"/>
 </segment>
 <segment>
@@
 <wire x1="137.16" y1="121.92" x2="134.62" y2="121.92" width="0.1524" layer="91"/>
 <label x="134.62" y="121.92" size="1.27" layer="95" font="vector" ratio="10" rot="R180" xref="yes"/>
-<pinref part="U1" gate="G$1" pin="/CS"/>
+<pinref part="U1" gate="G$1" pin="!CS"/>
 </segment>
 <segment>
@@
 <wire x1="137.16" y1="119.38" x2="134.62" y2="119.38" width="0.1524" layer="91"/>
 <label x="134.62" y="119.38" size="1.27" layer="95" font="vector" ratio="10" rot="R180" xref="yes"/>
-<pinref part="U1" gate="G$1" pin="/RES"/>
+<pinref part="U1" gate="G$1" pin="!RST"/>
 </segment>
 <segment>
@@
 </sheet>
 </sheets>
+<errors>
+</errors>
 </schematic>
 </drawing>
