File: pcb/Ai_Breakout_OLED-0.96.brd (EAGLE design)
At the start: 33 x 33 mm, 14 parts, among them J1 2X04, M1 STAND-OFF, M2 STAND-OFF, M3 STAND-OFF, M4 STAND-OFF, U1 UG-2864HSWEG01

Commit message: routing done
Parts:
- removed JP1: 1X07, Ai_Connectors:1X07
- added C1, C2: 10uF, Ai_Passives:CAP-0603
- added IC1: 74HCT245MTC, Ai_IC:SSOP20
- added J2: 1X08, Ai_Connectors:1X08
- added JS1, JS2: 1X02-SJ-NO, Ai_Connectors:1X02-SJ-NO
- added R1: 10K, Ai_Passives:RES-0603
- added U2: MIC5205-3.3, Ai_Power:SOT23-5
- C5: value 10uF -> 2.2uF
- C8: value 2.2uF -> 10uF
- moved C5 16.4 mm to (10.5, 16.1)
- moved C7 10.3 mm to (25.1, 16.1)
- moved C8 3.96 mm to (26.8, 16.1)
- moved R3 3.49 mm to (23.5, 16.1)
- moved C4 3.42 mm to (8.38, 16.1)
- moved C3 3.24 mm to (6.22, 16.1)
- moved C6 2.96 mm to (12.2, 16.1)
- moved J1 0.64 mm to (16.5, 30.5), flipped to the bottom
- moved U1 0.13 mm to (16.5, 13.2)
Connections:
- new net CS_IN: IC1.6, J1.5, J2.5
- new net D0/SCLK/SCK_IN: IC1.3, J1.2, J2.2
- new net D1/MOSI/SDA1_IN: IC1.2, J1.1, J2.1
- new net DC/SA0_IN: IC1.4, J1.3, J2.3
- new net I2C_EN: JS2.1, R1.2, U1.11
- new net N$8: JS1.2, U1.20
- new net RST_IN: IC1.5, J1.4, J2.4
- new net VIN: C1.2, J1.7, J2.7, U2.1, U2.3
- net 3V3: now also C2.2, C5.2, IC1.1, IC1.20, J1.6, J2.6, JS2.2, U2.5; no longer C7.2, JP1.6
- net CS_3V3: now also IC1.14; no longer JP1.5
- net D0/SCLK/SCK_3V3: now also IC1.17; no longer JP1.2
- net D1/MOSI/SDA1_3V3: now also IC1.18, JS1.1; no longer JP1.1
- net DC/SA0_3V3: now also IC1.16; no longer JP1.3
- net GND: now also C1.1, C2.1, IC1.10, IC1.19, J1.8, J2.8, R1.1, U2.2; no longer JP1.7, U1.11
- net N$11: now also C8.2; no longer C5.2
- net N$12: now also C7.2; no longer C8.2
- net RST_3V3: now also IC1.15; no longer JP1.4
Routing:
- net 3V3: track 0.00 -> 66.5 mm, vias 0 -> 2
- net DC/SA0_IN: track 0.00 -> 30.3 mm
- net RST_IN: track 0.00 -> 30.0 mm
- net CS_IN: track 0.00 -> 23.7 mm
- net D1/MOSI/SDA1_IN: track 0.00 -> 23.3 mm
- net D0/SCLK/SCK_IN: track 0.00 -> 21.5 mm
- net VIN: track 0.00 -> 20.3 mm
- net DC/SA0_3V3: track 0.00 -> 16.2 mm, vias 0 -> 2
- net D0/SCLK/SCK_3V3: track 0.00 -> 16.0 mm, vias 0 -> 2
- net CS_3V3: track 0.00 -> 14.4 mm
- net RST_3V3: track 0.00 -> 13.2 mm
- net D1/MOSI/SDA1_3V3: track 0.00 -> 10.7 mm
- net I2C_EN: track 0.00 -> 7.01 mm
- net N$7: track 0.00 -> 6.07 mm
- net N$5: track 0.00 -> 5.74 mm
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Other:
- board text removed: "1"
- board text removed: "10"
- board text removed: "20"
- board text removed: "30"

Commit message: ready for fabrication
Parts:
- added U$15, U$16: AI-LOGOXS, Ai_Miscellany:AI-LOGO-XS
- moved JS2 0.95 mm to (16.0, 17.3)
- moved JS1 0.57 mm to (19.6, 17.3), turned to 90 degrees
- moved U2 0.25 mm to (6.86, 29.6)
- moved IC1 0.13 mm to (16.6, 22.4)
- flipped J2 to the bottom
Routing:
- net D0/SCLK/SCK_IN: track 21.5 -> 41.9 mm, vias 0 -> 1
- net D1/MOSI/SDA1_IN: track 23.3 -> 39.7 mm, vias 0 -> 1
- net 3V3: track 66.5 -> 74.0 mm
- net N$8: track 4.79 -> 7.10 mm
- net D0/SCLK/SCK_3V3: track 16.0 -> 17.6 mm
- net DC/SA0_3V3: track 16.2 -> 17.8 mm
- net I2C_EN: track 7.01 -> 6.25 mm
- net D1/MOSI/SDA1_3V3: track 10.7 -> 11.4 mm
Other:
- board text added: "3V3"
- board text added: "D/C"
- board text added: "O: SPI C: I2C"
- board text added: "Pasadena, CA"
- board text added: "UG-2864HSWEG01 BREAKOUT"
- board text added: "VIN"
- board text added: "v1.0"
- board text removed: "3.3V"
- board text removed: "D/C#"
- board text removed: "SSD1306 1.3" 128x64 OLED"

Commit message: ready for manufacturing
Parts:
- moved C1 0.38 mm to (9.27, 29.7)
Other:
- board text added: "1"
- board text added: "2"
- board text added: "7"
- board text added: "8"
Changed lines of the file:
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@@
 <text x="5.334" y="9.652" size="1.016" layer="22" ratio="10" rot="MR0">SCK</text>
 <text x="5.969" y="7.112" size="1.016" layer="22" ratio="10" rot="MR0">SDIN</text>
-<text x="30.48" y="26.289" size="1.27" layer="22" ratio="10" rot="MR0">UG-2864HSWEG01 BREAKOUT</text>
+<text x="29.845" y="26.289" size="1.27" layer="22" ratio="10" rot="MR0">UG-2864HSWEG01 BREAKOUT</text>
 <text x="5.334" y="12.192" size="1.016" layer="22" ratio="10" rot="MR0">D/C</text>
 <rectangle x1="0" y1="0" x2="35" y2="35.5" layer="222"/>
@@
 <text x="19.177" y="16.256" size="0.6604" layer="22" font="vector" ratio="10" rot="MR180" align="bottom-right">O: SPI
 C: I2C</text>
+<text x="22.606" y="28.702" size="1.016" layer="22" ratio="10" rot="MR0">1</text>
+<text x="11.049" y="31.369" size="1.016" layer="22" ratio="10" rot="MR0">8</text>
+<text x="1.524" y="5.08" size="1.016" layer="22" ratio="10" rot="MR0">1</text>
+<text x="1.651" y="26.924" size="1.016" layer="22" ratio="10" rot="MR0">8</text>
+<text x="22.606" y="31.242" size="1.016" layer="22" ratio="10" rot="MR0">2</text>
+<text x="11.049" y="28.702" size="1.016" layer="22" ratio="10" rot="MR0">7</text>
 </plain>
 <attributes>
@@
 <attribute name="NAME" x="17.2212" y="16.002" size="1.27" layer="52" font="vector" ratio="15" rot="MR90"/>
 </element>
-<element name="U2" library="Ai_Power" package="SOT23-5" value="MIC5205-3.3" x="6.858" y="29.591" rot="MR180"/>
-<element name="C1" library="Ai_Passives" package="CAP-0603" value="10uF" x="9.652" y="29.718" smashed="yes" rot="MR90">
-<attribute name="NAME" x="9.271" y="31.496" size="0.8128" layer="26" font="vector" ratio="10" rot="MR90"/>
+<element name="U2" library="Ai_Power" package="SOT23-5" value="MIC5205-3.3" x="6.858" y="29.591" smashed="yes" rot="MR180">
+<attribute name="NAME" x="5.969" y="32.639" size="0.8128" layer="26" font="vector" ratio="10" rot="MR180"/>
+</element>
+<element name="C1" library="Ai_Passives" package="CAP-0603" value="10uF" x="9.271" y="29.718" smashed="yes" rot="MR90">
+<attribute name="NAME" x="8.89" y="31.496" size="0.8128" layer="26" font="vector" ratio="10" rot="MR90"/>
 </element>
 <element name="C2" library="Ai_Passives" package="CAP-0603" value="10uF" x="21.717" y="16.129" smashed="yes" rot="MR90">
@@
 <via x="28.194" y="24.892" extent="1-16" drill="0.381"/>
 <wire x1="17.272" y1="24.511" x2="13.637" y2="25.277" width="0" layer="19" extent="16-16"/>
-<wire x1="9.652" y1="28.818" x2="12.7" y2="31.75" width="0" layer="19" extent="16-16"/>
+<wire x1="9.271" y1="28.818" x2="12.7" y2="31.75" width="0" layer="19" extent="16-16"/>
 <wire x1="19.637" y1="20.077" x2="23.495" y2="17.029" width="0" layer="19" extent="16-16"/>
 <wire x1="14.1986" y1="17.029" x2="14.06" y2="12.008" width="0" layer="19" extent="16-16"/>
@@
 <wire x1="7.808" y1="30.8911" x2="7.808" y2="31.689" width="0.4064" layer="16"/>
 <wire x1="7.808" y1="30.8911" x2="9.3789" y2="30.8911" width="0.4064" layer="16"/>
-<wire x1="9.3789" y1="30.8911" x2="9.652" y2="30.618" width="0.4064" layer="16"/>
+<wire x1="9.3789" y1="30.8911" x2="9.271" y2="30.618" width="0.4064" layer="16"/>
 <wire x1="1.27" y1="22.86" x2="2.794" y2="22.86" width="0.4064" layer="16"/>
 <wire x1="2.794" y1="22.86" x2="5.08" y2="25.146" width="0.4064" layer="16"/>
@@
 <wire x1="12.7" y1="29.21" x2="11.303" y2="30.607" width="0.4064" layer="16"/>
 <wire x1="11.303" y1="30.607" x2="9.663" y2="30.607" width="0.4064" layer="16"/>
-<wire x1="9.663" y1="30.607" x2="9.652" y2="30.618" width="0.4064" layer="16"/>
+<wire x1="9.663" y1="30.607" x2="9.271" y2="30.618" width="0.4064" layer="16"/>
 </signal>
 <signal name="N$8">
