File: pcb/ai_breakout_oled-0.96.brd (EAGLE design)
At the start: 33 x 33 mm, 23 parts, among them IC1 74HCT245MTC, J1 2X04, J2 1X08, M1 STAND-OFF, M2 STAND-OFF, M3 STAND-OFF, M4 STAND-OFF, U1 UG-2864HSWEG01, U2 MIC5205-3.3

Commit message: Adding BOM.  Minor silkscreen changes
Parts:
- removed U2: MIC5205-3.3, Ai_Power:SOT23-5
- added OLED1: UG-2864HSWEG01, Ai_Displays:UG-2864HSWEG01_0.96_WRAP
- U1: value UG-2864HSWEG01 -> MIC5205-3.3; device Ai_Displays:UG-2864HSWEG01_0.96_WRAP -> Ai_Power:SOT23-5
- moved U1 19.0 mm to (6.86, 29.6), flipped to the bottom, turned to 180 degrees
- renumbered R3 to R2
Connections:
- net 3V3: now also OLED1.6, OLED1.9, U1.5; no longer U1.6, U1.9, U2.5
- net CS_3V3: now also OLED1.13; no longer U1.13
- net D0/SCLK/SCK_3V3: now also OLED1.18; no longer U1.18
- net D1/MOSI/SDA1_3V3: now also OLED1.19; no longer U1.19
- net DC/SA0_3V3: now also OLED1.15; no longer U1.15
- net GND: now also OLED1.1, OLED1.10, OLED1.12, OLED1.16, OLED1.17, OLED1.21, OLED1.22, OLED1.23, OLED1.24, OLED1.25, OLED1.29, OLED1.30, OLED1.8, U1.2; no longer U1.1, U1.10, U1.12, U1.16, U1.17, U1.21, U1.22, U1.23, U1.24, U1.25, U1.29, U1.30, U1.8, U2.2
- net I2C_EN: now also OLED1.11; no longer U1.11
- net N$11: now also OLED1.28; no longer U1.28
- net N$12: now also OLED1.27; no longer U1.27
- net N$3: now also OLED1.26; no longer U1.26
- net N$4: now also OLED1.2; no longer U1.2
- net N$5: now also OLED1.3; no longer U1.3
- net N$6: now also OLED1.4; no longer U1.4
- net N$7: now also OLED1.5; no longer U1.5
- net N$8: now also OLED1.20; no longer U1.20
- net RST_3V3: now also OLED1.14; no longer U1.14
- net VIN: now also U1.1, U1.3; no longer U2.1, U2.3
Changed lines of the file:
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@@
 <?xml version="1.0" encoding="utf-8"?>
 <!DOCTYPE eagle SYSTEM "eagle.dtd">
-<eagle version="6.5.0">
+<eagle version="7.1.0">
 <drawing>
 <settings>
@@
 <setting verticaltext="up"/>
 </settings>
-<grid distance="5" unitdist="mil" unit="mil" style="lines" multiple="1" display="yes" altdistance="0.025" altunitdist="inch" altunit="inch"/>
+<grid distance="50" unitdist="mil" unit="mil" style="lines" multiple="1" display="yes" altdistance="0.025" altunitdist="inch" altunit="inch"/>
 <layers>
 <layer number="1" name="Top" color="4" fill="1" visible="yes" active="yes"/>
@@
 <layer number="56" name="wert" color="7" fill="1" visible="no" active="yes"/>
 <layer number="57" name="tCAD" color="7" fill="1" visible="no" active="no"/>
-<layer number="90" name="Modules" color="5" fill="1" visible="yes" active="yes"/>
+<layer number="90" name="Modules" color="5" fill="1" visible="no" active="no"/>
 <layer number="91" name="Nets" color="2" fill="1" visible="no" active="no"/>
 <layer number="92" name="Busses" color="1" fill="1" visible="no" active="no"/>
@@
 <pass name="Default">
 <param name="RoutingGrid" value="50mil"/>
+<param name="AutoGrid" value="1"/>
+<param name="Efforts" value="0"/>
+<param name="TopRouterVariant" value="1"/>
 <param name="tpViaShape" value="round"/>
 <param name="PrefDir.1" value="|"/>
@@
 </autorouter>
 <elements>
-<element name="U1" library="Ai_Displays" package="UG-2864HSWEG01_0.96_WRAP" value="UG-2864HSWEG01" x="16.51" y="13.208" smashed="yes"/>
-<element name="R3" library="Ai_Passives" package="RES-0603" value="390K" x="23.495" y="16.129" smashed="yes" rot="MR270">
+<element name="OLED1" library="Ai_Displays" package="UG-2864HSWEG01_0.96_WRAP" value="UG-2864HSWEG01" x="16.51" y="13.208" smashed="yes"/>
+<element name="R2" library="Ai_Passives" package="RES-0603" value="390K" x="23.495" y="16.129" smashed="yes" rot="MR270">
 <attribute name="NAME" x="23.876" y="19.304" size="0.8128" layer="26" font="vector" ratio="10" rot="MR270"/>
 </element>
@@
 <attribute name="NAME" x="17.2212" y="16.002" size="1.27" layer="52" font="vector" ratio="15" rot="MR90"/>
 </element>
-<element name="U2" library="Ai_Power" package="SOT23-5" value="MIC5205-3.3" x="6.858" y="29.591" smashed="yes" rot="MR180">
+<element name="U1" library="Ai_Power" package="SOT23-5" value="MIC5205-3.3" x="6.858" y="29.591" smashed="yes" rot="MR180">
 <attribute name="NAME" x="5.969" y="32.639" size="0.8128" layer="26" font="vector" ratio="10" rot="MR180"/>
 </element>
@@
 <signals>
 <signal name="D0/SCLK/SCK_3V3">
-<contactref element="U1" pad="18"/>
+<contactref element="OLED1" pad="18"/>
 <contactref element="IC1" pad="17"/>
 <wire x1="18.26" y1="12.008" x2="18.26" y2="13.998" width="0.4064" layer="16"/>
@@
 </signal>
 <signal name="D1/MOSI/SDA1_3V3">
-<contactref element="U1" pad="19"/>
+<contactref element="OLED1" pad="19"/>
 <contactref element="JS1" pad="1"/>
 <contactref element="IC1" pad="18"/>
@@
 </signal>
 <signal name="GND" airwireshidden="yes">
-<contactref element="U1" pad="30"/>
-<contactref element="U1" pad="29"/>
-<contactref element="R3" pad="1"/>
+<contactref element="OLED1" pad="30"/>
+<contactref element="OLED1" pad="29"/>
+<contactref element="R2" pad="1"/>
 <contactref element="C8" pad="1"/>
 <contactref element="C7" pad="1"/>
@@
 <vertex x="33.02" y="0"/>
 </polygon>
-<contactref element="U1" pad="16"/>
-<contactref element="U1" pad="17"/>
-<contactref element="U1" pad="12"/>
-<contactref element="U1" pad="10"/>
-<contactref element="U1" pad="22"/>
-<contactref element="U1" pad="21"/>
-<contactref element="U1" pad="23"/>
-<contactref element="U1" pad="24"/>
-<contactref element="U1" pad="25"/>
-<contactref element="U1" pad="8"/>
+<contactref element="OLED1" pad="16"/>
+<contactref element="OLED1" pad="17"/>
+<contactref element="OLED1" pad="12"/>
+<contactref element="OLED1" pad="10"/>
+<contactref element="OLED1" pad="22"/>
+<contactref element="OLED1" pad="21"/>
+<contactref element="OLED1" pad="23"/>
+<contactref element="OLED1" pad="24"/>
+<contactref element="OLED1" pad="25"/>
+<contactref element="OLED1" pad="8"/>
 <contactref element="C6" pad="1"/>
 <contactref element="C5" pad="1"/>
-<contactref element="U1" pad="1"/>
+<contactref element="OLED1" pad="1"/>
 <contactref element="J2" pad="8"/>
 <contactref element="J1" pad="8"/>
 <contactref element="R1" pad="1"/>
-<contactref element="U2" pad="2"/>
+<contactref element="U1" pad="2"/>
 <contactref element="C1" pad="1"/>
 <contactref element="C2" pad="1"/>
@@
 </signal>
 <signal name="CS_3V3">
-<contactref element="U1" pad="13"/>
+<contactref element="OLED1" pad="13"/>
 <contactref element="IC1" pad="14"/>
 <wire x1="14.76" y1="12.008" x2="14.76" y2="13.998" width="0.4064" layer="16"/>
@@
 </signal>
 <signal name="RST_3V3">
-<contactref element="U1" pad="14"/>
+<contactref element="OLED1" pad="14"/>
 <contactref element="IC1" pad="15"/>
 <wire x1="15.46" y1="12.008" x2="15.46" y2="13.682" width="0.4064" layer="16"/>
@@
 </signal>
 <signal name="DC/SA0_3V3">
-<contactref element="U1" pad="15"/>
+<contactref element="OLED1" pad="15"/>
 <contactref element="IC1" pad="16"/>
 <wire x1="16.16" y1="12.008" x2="16.16" y2="13.2136" width="0.4064" layer="16"/>
@@
 </signal>
 <signal name="N$3">
-<contactref element="U1" pad="26"/>
-<contactref element="R3" pad="2"/>
+<contactref element="OLED1" pad="26"/>
+<contactref element="R2" pad="2"/>
 <wire x1="23.86" y1="12.008" x2="23.86" y2="14.864" width="0.4064" layer="16"/>
 <wire x1="23.86" y1="14.864" x2="23.495" y2="15.229" width="0.4064" layer="16"/>
 </signal>
 <signal name="N$4">
-<contactref element="U1" pad="2"/>
+<contactref element="OLED1" pad="2"/>
 <contactref element="C3" pad="2"/>
 <wire x1="7.06" y1="12.008" x2="7.06" y2="13.26" width="0.4064" layer="16"/>
@@
 <signal name="N$5">
 <contactref element="C3" pad="1"/>
-<contactref element="U1" pad="3"/>
+<contactref element="OLED1" pad="3"/>
 <wire x1="7.76" y1="12.008" x2="7.76" y2="13.703" width="0.4064" layer="16"/>
 <wire x1="7.76" y1="13.703" x2="7.239" y2="14.224" width="0.4064" layer="16"/>
@@
 </signal>
 <signal name="N$6">
-<contactref element="U1" pad="4"/>
+<contactref element="OLED1" pad="4"/>
 <contactref element="C4" pad="2"/>
 <wire x1="8.46" y1="12.008" x2="8.46" y2="15.151" width="0.4064" layer="16"/>
@@
 <signal name="N$7">
 <contactref element="C4" pad="1"/>
-<contactref element="U1" pad="5"/>
+<contactref element="OLED1" pad="5"/>
 <wire x1="8.382" y1="17.029" x2="9.26" y2="17.029" width="0.4064" layer="16"/>
 <wire x1="9.26" y1="17.029" x2="9.398" y2="16.891" width="0.4064" layer="16"/>
@@
 </signal>
 <signal name="N$11">
-<contactref element="U1" pad="28"/>
+<contactref element="OLED1" pad="28"/>
 <contactref element="C8" pad="2"/>
 <wire x1="25.26" y1="12.008" x2="25.26" y2="13.703" width="0.4064" layer="16"/>
@@
 </signal>
 <signal name="N$12">
-<contactref element="U1" pad="27"/>
+<contactref element="OLED1" pad="27"/>
 <contactref element="C7" pad="2"/>
 <wire x1="24.56" y1="12.008" x2="24.56" y2="14.643" width="0.4064" layer="16"/>
@@
 </signal>
 <signal name="3V3">
-<contactref element="U1" pad="6"/>
+<contactref element="OLED1" pad="6"/>
 <contactref element="C5" pad="2"/>
-<contactref element="U1" pad="9"/>
+<contactref element="OLED1" pad="9"/>
 <contactref element="C6" pad="2"/>
 <contactref element="J2" pad="6"/>
@@
 <contactref element="JS2" pad="2"/>
 <contactref element="C2" pad="2"/>
-<contactref element="U2" pad="5"/>
+<contactref element="U1" pad="5"/>
 <contactref element="IC1" pad="20"/>
 <contactref element="IC1" pad="1"/>
@@
 <contactref element="J2" pad="7"/>
 <contactref element="J1" pad="7"/>
-<contactref element="U2" pad="1"/>
+<contactref element="U1" pad="1"/>
 <contactref element="C1" pad="2"/>
-<contactref element="U2" pad="3"/>
+<contactref element="U1" pad="3"/>
 <wire x1="5.908" y1="30.8911" x2="5.908" y2="31.689" width="0.4064" layer="16"/>
 <wire x1="5.908" y1="31.689" x2="6.223" y2="32.004" width="0.4064" layer="16"/>
@@
 <signal name="N$8">
 <contactref element="JS1" pad="2"/>
-<contactref element="U1" pad="20"/>
+<contactref element="OLED1" pad="20"/>
 <wire x1="19.66" y1="12.008" x2="19.66" y2="14.859" width="0.4064" layer="16"/>
 <wire x1="19.66" y1="14.859" x2="19.66" y2="15.781" width="0" layer="19" extent="1-16"/>
@@
 </signal>
 <signal name="I2C_EN">
-<contactref element="U1" pad="11"/>
+<contactref element="OLED1" pad="11"/>
 <contactref element="JS2" pad="1"/>
 <contactref element="R1" pad="2"/>
